File: MMS3/MMS_CONNECTOR.kicad_sch (KiCad schematic)
At the start: 6 parts, among them J8 RJ45_LED_Shielded, U4 TPD2EUSB30DRTR-TP

Commit message: updated schematic, removed annotation
Other:
- title: MMS3 -> MMS3 CH32L103 Version
Changed lines of the file:
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@@
 	(paper "A4")
 	(title_block
-		(title "MMS3")
-		(date "2026-04-03")
+		(title "MMS3 CH32L103 Version")
+		(date "2026-05-18")
 		(rev "XA1")
 		(company "(c) Modular Mechanica")
-		(comment 1 "Artem Horiunov")
-		(comment 2 "DESIGNED IN POLAND")
+		(comment 1 "DESIGNED IN POLAND")
+		(comment 2 "Forked by: Wojciech Szafranski")
+		(comment 3 "Made by: Artem Horiunov")
 	)
 	(junction
