File: MMS3/PSU.kicad_sch (KiCad schematic)
At the start: 19 parts, among them U15 AMS1117-3.3

Commit message: initial PCB update
Parts:
- gave numbers to parts that had none: 14
Changed lines of the file:
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@@
 		(dnp no)
 		(fields_autoplaced yes)
-		(property "Reference" "R?"
+		(property "Reference" "R18"
 			(at 147.32 175.2599 0)
 			(show_name no)
@@
 			(project "MMS3"
 				(path "/712cea22-140d-4c92-923f-f4998caf3ecd/9a06b27f-9b6a-4e31-92df-df3bedc6f86c"
-					(reference "R?")
+					(reference "R18")
 					(unit 1)
 				)
@@
 		(dnp no)
 		(fields_autoplaced yes)
-		(property "Reference" "D?"
+		(property "Reference" "D10"
 			(at 198.4375 91.1491 90)
 			(show_name no)
@@
 			(project "MMS3"
 				(path "/712cea22-140d-4c92-923f-f4998caf3ecd/9a06b27f-9b6a-4e31-92df-df3bedc6f86c"
-					(reference "D?")
+					(reference "D10")
 					(unit 1)
 				)
@@
 		(dnp no)
 		(fields_autoplaced yes)
-		(property "Reference" "#PWR?"
+		(property "Reference" "#PWR091"
 			(at 149.86 162.56 0)
 			(hide yes)
@@
 			(project "MMS3"
 				(path "/712cea22-140d-4c92-923f-f4998caf3ecd/9a06b27f-9b6a-4e31-92df-df3bedc6f86c"
-					(reference "#PWR?")
+					(reference "#PWR091")
 					(unit 1)
 				)
@@
 		(dnp no)
 		(fields_autoplaced yes)
-		(property "Reference" "C?"
+		(property "Reference" "C16"
 			(at 78.74 104.1399 0)
 			(show_name no)
@@
 			(project "MMS3"
 				(path "/712cea22-140d-4c92-923f-f4998caf3ecd/9a06b27f-9b6a-4e31-92df-df3bedc6f86c"
-					(reference "C?")
+					(reference "C16")
 					(unit 1)
 				)
@@
 		(dnp no)
 		(fields_autoplaced yes)
-		(property "Reference" "R?"
+		(property "Reference" "R19"
 			(at 168.91 119.3799 0)
 			(show_name no)
@@
 			(project "MMS3"
 				(path "/712cea22-140d-4c92-923f-f4998caf3ecd/9a06b27f-9b6a-4e31-92df-df3bedc6f86c"
-					(reference "R?")
+					(reference "R19")
 					(unit 1)
 				)
@@
 		(dnp no)
 		(fields_autoplaced yes)
-		(property "Reference" "#PWR?"
+		(property "Reference" "#PWR094"
 			(at 182.88 121.92 0)
 			(hide yes)
@@
 			(project "MMS3"
 				(path "/712cea22-140d-4c92-923f-f4998caf3ecd/9a06b27f-9b6a-4e31-92df-df3bedc6f86c"
-					(reference "#PWR?")
+					(reference "#PWR094")
 					(unit 1)
 				)
@@
 		(dnp no)
 		(fields_autoplaced yes)
-		(property "Reference" "#PWR?"
+		(property "Reference" "#PWR092"
 			(at 149.86 186.69 0)
 			(hide yes)
@@
 			(project "MMS3"
 				(path "/712cea22-140d-4c92-923f-f4998caf3ecd/9a06b27f-9b6a-4e31-92df-df3bedc6f86c"
-					(reference "#PWR?")
+					(reference "#PWR092")
 					(unit 1)
 				)
@@
 		(dnp no)
 		(fields_autoplaced yes)
-		(property "Reference" "C?"
+		(property "Reference" "C18"
 			(at 185.42 104.1399 0)
 			(show_name no)
@@
 			(project "MMS3"
 				(path "/712cea22-140d-4c92-923f-f4998caf3ecd/9a06b27f-9b6a-4e31-92df-df3bedc6f86c"
-					(reference "C?")
+					(reference "C18")
 					(unit 1)
 				)
@@
 		(dnp no)
 		(fields_autoplaced yes)
-		(property "Reference" "C?"
+		(property "Reference" "C19"
 			(at 257.81 67.6909 0)
 			(show_name no)
@@
 			(project "MMS3"
 				(path "/712cea22-140d-4c92-923f-f4998caf3ecd/9a06b27f-9b6a-4e31-92df-df3bedc6f86c"
-					(reference "C?")
+					(reference "C19")
 					(unit 1)
 				)
@@
 		(dnp no)
 		(fields_autoplaced yes)
-		(property "Reference" "R?"
+		(property "Reference" "R20"
 			(at 168.91 137.1599 0)
 			(show_name no)
@@
 			(project "MMS3"
 				(path "/712cea22-140d-4c92-923f-f4998caf3ecd/9a06b27f-9b6a-4e31-92df-df3bedc6f86c"
-					(reference "R?")
+					(reference "R20")
 					(unit 1)
 				)
@@
 		(dnp no)
 		(fields_autoplaced yes)
-		(property "Reference" "R?"
+		(property "Reference" "R16"
 			(at 91.44 58.4199 0)
 			(show_name no)
@@
 			(project "MMS3"
 				(path "/712cea22-140d-4c92-923f-f4998caf3ecd/9a06b27f-9b6a-4e31-92df-df3bedc6f86c"
-					(reference "R?")
+					(reference "R16")
 					(unit 1)
 				)
@@
 		(dnp no)
 		(fields_autoplaced yes)
-		(property "Reference" "#PWR?"
+		(property "Reference" "#PWR096"
 			(at 254 107.95 0)
 			(hide yes)
@@
 			(project "MMS3"
 				(path "/712cea22-140d-4c92-923f-f4998caf3ecd/9a06b27f-9b6a-4e31-92df-df3bedc6f86c"
-					(reference "#PWR?")
+					(reference "#PWR096")
 					(unit 1)
 				)
@@
 		(dnp no)
 		(fields_autoplaced yes)
-		(property "Reference" "#PWR?"
+		(property "Reference" "#PWR095"
 			(at 232.41 107.95 0)
 			(hide yes)
@@
 			(project "MMS3"
 				(path "/712cea22-140d-4c92-923f-f4998caf3ecd/9a06b27f-9b6a-4e31-92df-df3bedc6f86c"
-					(reference "#PWR?")
+					(reference "#PWR095")
 					(unit 1)
 				)
@@
 		(dnp no)
 		(fields_autoplaced yes)
-		(property "Reference" "C?"
+		(property "Reference" "C17"
 			(at 153.67 119.3799 0)
 			(show_name no)
@@
 			(project "MMS3"
 				(path "/712cea22-140d-4c92-923f-f4998caf3ecd/9a06b27f-9b6a-4e31-92df-df3bedc6f86c"
-					(reference "C?")
+					(reference "C17")
 					(unit 1)
 				)
@@
 		(dnp no)
 		(fields_autoplaced yes)
-		(property "Reference" "D?"
+		(property "Reference" "D9"
 			(at 154.94 165.0046 0)
 			(show_name no)
@@
 			(project "MMS3"
 				(path "/712cea22-140d-4c92-923f-f4998caf3ecd/9a06b27f-9b6a-4e31-92df-df3bedc6f86c"
-					(reference "D?")
+					(reference "D9")
 					(unit 1)
 				)
@@
 		(dnp no)
 		(fields_autoplaced yes)
-		(property "Reference" "#PWR?"
+		(property "Reference" "#PWR082"
 			(at 76.2 123.19 0)
 			(hide yes)
@@
 			(project "MMS3"
 				(path "/712cea22-140d-4c92-923f-f4998caf3ecd/9a06b27f-9b6a-4e31-92df-df3bedc6f86c"
-					(reference "#PWR?")
+					(reference "#PWR082")
 					(unit 1)
 				)
@@
 		(dnp no)
 		(fields_autoplaced yes)
-		(property "Reference" "#PWR?"
+		(property "Reference" "#PWR097"
 			(at 260.35 57.15 0)
 			(hide yes)
@@
 			(project "MMS3"
 				(path "/712cea22-140d-4c92-923f-f4998caf3ecd/9a06b27f-9b6a-4e31-92df-df3bedc6f86c"
-					(reference "#PWR?")
+					(reference "#PWR097")
 					(unit 1)
 				)
@@
 		(dnp no)
 		(fields_autoplaced yes)
-		(property "Reference" "D?"
+		(property "Reference" "D8"
 			(at 137.16 165.0046 0)
 			(show_name no)
@@
 			(project "MMS3"
 				(path "/712cea22-140d-4c92-923f-f4998caf3ecd/9a06b27f-9b6a-4e31-92df-df3bedc6f86c"
-					(reference "D?")
+					(reference "D8")
 					(unit 1)
 				)
@@
 		(dnp no)
 		(fields_autoplaced yes)
-		(property "Reference" "#PWR?"
+		(property "Reference" "#PWR083"
 			(at 88.9 71.12 0)
 			(hide yes)
@@
 			(project "MMS3"
 				(path "/712cea22-140d-4c92-923f-f4998caf3ecd/9a06b27f-9b6a-4e31-92df-df3bedc6f86c"
-					(reference "#PWR?")
+					(reference "#PWR083")
 					(unit 1)
 				)
@@
 		(dnp no)
 		(fields_autoplaced yes)
-		(property "Reference" "#PWR?"
+		(property "Reference" "#PWR093"
 			(at 166.37 149.86 0)
 			(hide yes)
@@
 			(project "MMS3"
 				(path "/712cea22-140d-4c92-923f-f4998caf3ecd/9a06b27f-9b6a-4e31-92df-df3bedc6f86c"
-					(reference "#PWR?")
+					(reference "#PWR093")
 					(unit 1)
 				)
@@
 		(dnp no)
 		(fields_autoplaced yes)
-		(property "Reference" "#PWR?"
+		(property "Reference" "#PWR090"
 			(at 132.08 186.69 0)
 			(hide yes)
@@
 			(project "MMS3"
 				(path "/712cea22-140d-4c92-923f-f4998caf3ecd/9a06b27f-9b6a-4e31-92df-df3bedc6f86c"
-					(reference "#PWR?")
+					(reference "#PWR090")
 					(unit 1)
 				)
@@
 		(dnp no)
 		(fields_autoplaced yes)
-		(property "Reference" "U?"
+		(property "Reference" "U7"
 			(at 130.81 116.84 0)
 			(show_name no)
@@
 			(project "MMS3"
 				(path "/712cea22-140d-4c92-923f-f4998caf3ecd/9a06b27f-9b6a-4e31-92df-df3bedc6f86c"
-					(reference "U?")
+					(reference "U7")
 					(unit 1)
 				)
@@
 		(dnp no)
 		(fields_autoplaced yes)
-		(property "Reference" "#PWR?"
+		(property "Reference" "#PWR088"
 			(at 132.08 162.56 0)
 			(hide yes)
@@
 			(project "MMS3"
 				(path "/712cea22-140d-4c92-923f-f4998caf3ecd/9a06b27f-9b6a-4e31-92df-df3bedc6f86c"
-					(reference "#PWR?")
+					(reference "#PWR088")
 					(unit 1)
 				)
@@
 		(dnp no)
 		(fields_autoplaced yes)
-		(property "Reference" "#PWR?"
+		(property "Reference" "#PWR086"
 			(at 111.76 142.24 0)
 			(hide yes)
@@
 			(project "MMS3"
 				(path "/712cea22-140d-4c92-923f-f4998caf3ecd/9a06b27f-9b6a-4e31-92df-df3bedc6f86c"
-					(reference "#PWR?")
+					(reference "#PWR086")
 					(unit 1)
 				)
@@
 		(dnp no)
 		(fields_autoplaced yes)
-		(property "Reference" "R?"
+		(property "Reference" "R15"
 			(at 91.44 44.4499 0)
 			(show_name no)
@@
 			(project "MMS3"
 				(path "/712cea22-140d-4c92-923f-f4998caf3ecd/9a06b27f-9b6a-4e31-92df-df3bedc6f86c"
-					(reference "R?")
+					(reference "R15")
 					(unit 1)
 				)
@@
 		(dnp no)
 		(fields_autoplaced yes)
-		(property "Reference" "R?"
+		(property "Reference" "R17"
 			(at 134.62 175.2599 0)
 			(show_name no)
@@
 			(project "MMS3"
 				(path "/712cea22-140d-4c92-923f-f4998caf3ecd/9a06b27f-9b6a-4e31-92df-df3bedc6f86c"
-					(reference "R?")
+					(reference "R17")
 					(unit 1)
 				)
